File: OchlastaPCB/OchlastaPCB.kicad_sch (KiCad schematic)
At the start: 136 parts, among them J1 XT60PW-M, J2 5V, J3 Conn_01x02_Socket, Q1 IRFH7440, Q2 IRFH7440, U1 AP64501SP-13, U10 INA333xxDGK, U11 INA333xxDGK, U12 INA333xxDGK, U13 UCC27282DR, U14 AP64501SP-13, U2 AP3429, U3 STM32F334R8Tx, U4 INA333xxDGK, U5 TPS7A4901DGNR, U6 INA333xxDGK, U7 INA333xxDGK, U8 INA333xxDGK, U9 INA333xxDGK, Y1 Crystal_GND24

Commit message: Schematics done except for CAN transciever
Parts:
- removed U2: AP3429, Package_TO_SOT_SMD:TSOT-23-5, symbol Greels symbol library:AP3429
- removed U5: TPS7A4901DGNR, SnapMagic_downloads:SOP65P490X110-9N, symbol TPS7A4901DGNR:TPS7A4901DGNR
- added C45, C47, C52, C53, C56, C57, C66, C67, C68, C69, C70: 100 n, Capacitor_SMD:C_0603_1608Metric, symbol Device:C
- added C46, C54, C55: 1 u, Capacitor_SMD:C_0603_1608Metric, symbol Device:C
- added C48, C49, C50, C51, C58, C59, C60, C61, C62, C63, C64, C65: 10 uF 50V, Capacitor_SMD:C_1206_3216Metric, symbol Device:C
- added C71, C72, C73, C74: 100 n, symbol Device:C
- added CP4, CP5, CP6: 100 uF, Capacitor_SMD:CP_Elec_8x10, symbol Device:C_Polarized
- added D10, D11, D12, D13, D14, D15, D16, D5, D6, D7, D8, D9: SS14, Diode_SMD:D_SMA, symbol Device:D_Schottky
- added J4, J5, J6: Conn_01x02_Socket, TerminalBlock_WAGO:TerminalBlock_WAGO_236-402_1x02_P5.00mm_45Degree, symbol Connector:Conn_01x02_Socket
- added J7: Debug, symbol Connector_Generic:Conn_02x05_Odd_Even
- added J8: UART, symbol Connector:Conn_01x03_Pin
- added L5, L6, L7: 22 uH, Inductor_SMD:L_APV_APH1770, symbol Device:L
- added Q3, Q4, Q5, Q6, Q7, Q8: IRFH7440, SnapMagic_downloads:PQFN_5x6_FET, symbol Simulation_SPICE:NMOS
- added R20, R21, R22, R23, R24, R25, R26, R27, R28, R29, R30, R31: 10 R, Resistor_SMD:R_0603_1608Metric, symbol Device:R
- added R32, R33: 10k, Resistor_SMD:R_0603_1608Metric, symbol Device:R
- added R34, R36, R38, R40, R42: 200k 1%, Resistor_SMD:R_0603_1608Metric, symbol Device:R
- added R35, R37, R39, R41, R43: 22.1 k 1%, Resistor_SMD:R_0603_1608Metric, symbol Device:R
- added Rshunt1, Rshunt2, Rshunt3, Rshunt4: 5 mR, Resistor_SMD:R_1206_3216Metric, symbol Device:R
- added SW1: SW_RESET, symbol Switch:SW_SPST
- added SW2: SW_BOOT, symbol Switch:SW_SPST
- added U15, U16, U17: UCC27282DR, SnapMagic_downloads:SOIC127P599X175-8N, symbol UCC27282DR:UCC27282DR
- added U18, U19, U20, U21: INA240A2D, Package_SO:SOIC-8_3.9x4.9mm_P1.27mm, symbol Amplifier_Current:INA240A2D
- added U2: AP3429, Package_TO_SOT_SMD:TSOT-23-5, symbol OchlastaSymbols:AP3429
- added U5: TPS7A4901DGNR_Trafo_Edit, SnapMagic_downloads:SOP65P490X110-9N, symbol OchlastaSymbols:TPS7A4901DGNR_Trafo_Edit
Connections:
- net +3.3VA: now also U3.13 (VDDA), C70.1, C71.1, C72.1, C73.1, C74.1, U18.6 (V+), U19.6 (V+), U20.6 (V+), U21.6 (V+), U5.1 (OUT); no longer C16.1
- net +3V3: now also U3.1 (VBAT), U3.19 (VDD), U3.32 (VDD), U3.48 (VDD), U3.64 (VDD), C66.1, C67.1, C68.1, C69.1, J7.1 (Pin_1), SW2.1 (A)
- net +5V: now also U2.4 (VIN), U5.8 (IN)
- net +8V: now also C45.2, C46.2, C52.2, C53.2, C54.2, C55.2, U15.1 (VDD), U16.1 (VDD), U17.1 (VDD)
- net +vin: now also Q3.1 (D), Q5.1 (D), Q7.1 (D), R42.1
- net GND: now also C16.2, U3.12 (VSSA), U3.18 (VSS), U3.31 (VSS), U3.47 (VSS), U3.63 (VSS), C45.1, C46.1, C48.2, C49.2, C50.2, C51.2, C52.1, C53.1, C54.1, C55.1, C58.2, C59.2, C60.2, C61.2, C62.2, C63.2, C64.2, C65.2, C66.2, C67.2, C68.2, C69.2, C70.2, C71.2, C72.2, C73.2, C74.2, CP4.2, CP5.2, CP6.2, D11.2 (A), D12.2 (A), D6.2 (A), J4.1 (Pin_1), J5.1 (Pin_1), J6.1 (Pin_1), J7.3 (Pin_3), J7.5 (Pin_5), J7.9 (Pin_9), J8.1 (Pin_1), Q4.3 (S), Q6.3 (S), Q8.3 (S), R33.1, R35.2, R37.2, R39.2, R41.2, R43.2, SW1.1 (A), U15.7 (VSS), U16.7 (VSS), U17.7 (VSS), U18.2 (GND), U18.3 (REF2), U18.4 (GND), U18.7 (REF1), U19.2 (GND), U19.3 (REF2), U19.4 (GND), U19.7 (REF1), U2.2 (GND), U20.2 (GND), U20.3 (REF2), U20.4 (GND), U20.7 (REF1), U21.2 (GND), U21.3 (REF2), U21.4 (GND), U21.7 (REF1), U5.4 (GND), U5.9 (EP)
- net HRTIM_A_Hi: now also U3.41 (PA8)
- net HRTIM_A_Lo: now also U3.42 (PA9)
- net temp_U_out_1: now also U3.11 (PC3)
- net temp_U_out_2: now also U3.20 (PA4)
- net temp_U_out_3: now also U3.21 (PA5)
- net temp_U_out_4: now also U3.22 (PA6)
- net temp_U_out_5: now also U3.23 (PA7)
- net temp_U_out_6: now also U3.24 (PC4)
- net temp_U_out_7: now also U3.25 (PC5)
- net temp_U_out_8: now also U3.28 (PB2)
- net at C11.2, R6.2, R7.1: now also U2.5 (FB)
- net at C41.1, C42.1, C43.1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: now also Rshunt1.1, U18.8 (+); no longer J3.2 (Pin_2)
- net at R10.2, R11.1: now also C16.1, U5.2 (FB); no longer C16.2
- net at R9.2: now also U5.5 (EN)
- net at C19.1: now also U5.6 (NR/SS)
- net HSE_OUT: now reaches C17.1, Y1.1
- net HSE_OUT: now also U3.6 (PF1)
- net at R5.2: now also U2.1 (EN)
- net U_out_3: now reaches U3.10 (PC2)
- net U_out_3: now also R38.2, R39.1
- net I_out_1: now reaches U3.14 (PA0)
- net I_out_1: now also U18.5
- net I_out_2: now reaches U3.15 (PA1)
- net I_out_2: now also U19.5
- net I_out_3: now reaches U3.16 (PA2)
- net I_out_3: now also U20.5
- net I_out_4: now reaches U3.17 (PA3)
- net I_out_4: now also U21.5
- net U_out_4: now reaches U3.26 (PB0)
- net U_out_4: now also R40.2, R41.1
- net U_input_div: now reaches U3.27 (PB1)
- net U_input_div: now also R42.2, R43.1
- net PB10_Disp_RST: now reaches U3.29 (PB10)
- net PB10_Disp_RST: now also TFT1.5 (RST)
- net PB11_Disp_DC: now reaches U3.30 (PB11)
- net PB11_Disp_DC: now also TFT1.6 (DC)
- net HRTIM_C_Hi: now reaches U3.33 (PB12)
- net HRTIM_C_Hi: now also U16.5 (HI)
- net HRTIM_C_Lo: now reaches U3.34 (PB13)
- net HRTIM_C_Lo: now also U16.6 (LI)
- net HRTIM_D_Hi: now reaches U3.35 (PB14)
- net HRTIM_D_Hi: now also U17.5 (HI)
- net HRTIM_D_Lo: now reaches U3.36 (PB15)
- net HRTIM_D_Lo: now also U17.6 (LI)
- net HRTIM_B_Hi: now reaches U3.43 (PA10)
- net HRTIM_B_Hi: now also U15.5 (HI)
- net HRTIM_B_Lo: now reaches U3.44 (PA11)
- net HRTIM_B_Lo: now also U15.6 (LI)
- net CAN_TX: now reaches U3.45 (PA12)
- net SWDIO: now reaches U3.46 (PA13)
- net SWDIO: now also J7.2 (Pin_2)
- net SWCLK: now reaches U3.49 (PA14)
- net SWCLK: now also J7.4 (Pin_4)
- net HSE_IN: now reaches U3.5 (PF0)
- net HSE_IN: now also R8.1
- net SPI_SCK: now reaches U3.55 (PB3)
- net SPI_SCK: now also TFT1.3 (SCL)
- net SPI_MISO: now reaches U3.56 (PB4)
- net SPI_MOSI: now reaches U3.57 (PB5)
- net SPI_MOSI: now also TFT1.4 (SDA/MOSI)
- net UART_TX: now reaches U3.58 (PB6)
- net UART_TX: now also J8.2 (Pin_2)
- net UART_RX: now reaches U3.59 (PB7)
- net UART_RX: now also J8.3 (Pin_3)
- net BOOT0: now reaches U3.60 (BOOT0)
- net BOOT0: now also R32.2
- net CAN_RX: now reaches U3.61 (PB8)
- net PB9_Disp_CS: now reaches U3.62 (PB9)
- net PB9_Disp_CS: now also TFT1.7 (CS)
- net NRST: now reaches U3.7 (NRST)
- net NRST: now also J7.10 (Pin_10), SW1.2 (B)
- net U_out_1: now reaches U3.8 (PC0)
- net U_out_1: now also R34.2, R35.1
- net U_out_2: now reaches U3.9 (PC1)
- net U_out_2: now also R36.2, R37.1
- net at L2.1: now also U2.3 (LX)
- new net: D5.1 (K), D7.1 (K), R20.1, U15.3 (HO)
- new net: Q3.2 (G), R20.2, R22.2
- new net: D8.2 (A), R23.1
- new net: Q4.2 (G), R21.2, R23.2
- new net: C48.1, C49.1, C50.1, C51.1, CP4.1, L5.2, Rshunt2.1, U19.8 (+)
- new net: C59.1, C61.1, C63.1, C65.1, CP6.1, L7.2, Rshunt4.1, U21.8 (+)
- new net: D14.2 (A), R29.1
- new net: Q6.2 (G), R25.2, R29.2
- new net: D10.1 (K), D15.1 (K), R26.1, U17.3 (HO)
- new net: Q7.2 (G), R26.2, R30.2
- new net: C57.1, U17.2 (HB)
- new net: C57.2, D10.2 (A), L7.1, Q7.3 (S), Q8.1 (D), U17.4 (HS)
- new net: D12.1 (K), D16.1 (K), R27.1, U17.8 (LO)
- new net: J5.2 (Pin_2), R38.1, Rshunt3.2, U20.1 (-)
- new net: Q8.2 (G), R27.2, R31.2
- new net: D13.1 (K), D9.1 (K), R24.1, U16.3 (HO)
- new net: D13.2 (A), R28.1
- new net: D11.1 (K), D14.1 (K), R25.1, U16.8 (LO)
- new net: C56.2, D9.2 (A), L6.1, Q5.3 (S), Q6.1 (D), U16.4 (HS)
- new net: J3.2 (Pin_2), R34.1, Rshunt1.2, U18.1 (-)
- new net: J6.2 (Pin_2), R40.1, Rshunt4.2, U21.1 (-)
- new net: C47.2, D5.2 (A), L5.1, Q3.3 (S), Q4.1 (D), U15.4 (HS)
- new net: D6.1 (K), D8.1 (K), R21.1, U15.8 (LO)
- new net: J4.2 (Pin_2), R36.1, Rshunt2.2, U19.1 (-)
- new net: Q5.2 (G), R24.2, R28.2
- new net: D7.2 (A), R22.1
- new net: C58.1, C60.1, C62.1, C64.1, CP5.1, L6.2, Rshunt3.1, U20.8 (+)
- new net: C56.1, U16.2 (HB)
- new net: R32.1, R33.2, SW2.2 (B)
- new net: D15.2 (A), R30.1
- new net: C47.1, U15.2 (HB)
- new net: D16.2 (A), R31.1
- no-connect marks 1 -> 18
Other:
- note added: "Assume 10A, 5mOhm gives 0.05V lets use 50x amplification. That would result in 2.5V at 10A"
- note added: "Ground referenced output"
- moved on the sheet: C16, C17, C18, C20, C21, J3, R10, R11, R8, U3, Y1

Commit message: Schematics complete I guess
Parts:
- added C75: 100 n, Capacitor_SMD:C_0603_1608Metric, symbol Device:C
- added H1, H2, H3, H4: MountingHole_Pad, MountingHole:MountingHole_3.2mm_M3_Pad_Via, symbol Mechanical:MountingHole_Pad
- added J10: CAN term jmp, Connector_PinHeader_2.54mm:PinHeader_1x02_P2.54mm_Vertical, symbol Connector:Conn_01x02_Pin
- added J9: CAN, symbol Connector:Screw_Terminal_01x02
- added R44: 120 R, Resistor_SMD:R_0603_1608Metric, symbol Device:R
- added R45: 120 R / DNP, Resistor_SMD:R_0603_1608Metric, symbol Device:R
- added R46: DNP / 120 R, Resistor_SMD:R_0603_1608Metric, symbol Device:R
- added R47, R48, R49, R50, R51, R52, R53, R54, R55: 10 k, Resistor_SMD:R_0603_1608Metric, symbol Device:R
- added SW3: BTN_A, Button_Switch_THT:SW_PUSH_6mm, symbol Switch:SW_SPST
- added SW4: RotaryEncoder_Switch, Rotary_Encoder:RotaryEncoder_Alps_EC11E-Switch_Vertical_H20mm, symbol Device:RotaryEncoder_Switch
- added SW5: BTN_B, Button_Switch_THT:SW_PUSH_6mm, symbol Switch:SW_SPST
- added SW6: BTN_C, Button_Switch_THT:SW_PUSH_6mm, symbol Switch:SW_SPST
- added SW7: BTN_D, Button_Switch_THT:SW_PUSH_6mm, symbol Switch:SW_SPST
- added SW8: BTN_L, Button_Switch_THT:SW_PUSH_6mm, symbol Switch:SW_SPST
- added SW9: BTN_R, Button_Switch_THT:SW_PUSH_6mm, symbol Switch:SW_SPST
- added U22: SN65HVD230, Package_SO:SOIC-8_3.9x4.9mm_P1.27mm, symbol Interface_CAN_LIN:SN65HVD230
- C71, C72, C73, C74: footprint (none) -> Capacitor_SMD:C_0603_1608Metric
- J7: footprint (none) -> Connector_IDC:IDC-Header_2x05_P2.54mm_Vertical
- J8: footprint (none) -> Connector_PinHeader_2.54mm:PinHeader_1x03_P2.54mm_Vertical
- SW1, SW2: footprint (none) -> OchlastaFootprints:SW_Push_SPST_CheapAtJLC
Connections:
- net +3V3: now also C75.1, R45.1, R47.1, R48.1, R49.1, R50.1, R51.1, R52.1, R53.1, R54.1, R55.1, U22.3 (VCC)
- net CAN_RX: now also U22.1 (D)
- net CAN_TX: now also U22.4 (R)
- net GND: now also C75.2, H1.1, H2.1, H3.1, H4.1, R46.1, SW3.2 (B), SW4.C, SW4.S2, SW5.2 (B), SW6.2 (B), SW7.2 (B), SW8.2 (B), SW9.2 (B), U22.2 (GND)
- net BTN_L: now reaches U3.2 (PC13)
- net BTN_L: now also R52.2, SW8.1 (A)
- net BTN_R: now reaches U3.3 (PC14)
- net BTN_R: now also R51.2, SW9.1 (A)
- net ENC_A: now reaches U3.37 (PC6)
- net ENC_A: now also R54.2, SW4.A
- net ENC_B: now reaches U3.38 (PC7)
- net ENC_B: now also R53.2, SW4.B
- net BTN_ENC: now reaches U3.39 (PC8)
- net BTN_ENC: now also R55.2, SW4.S1
- net BTN_A: now reaches U3.40 (PC9)
- net BTN_A: now also R47.2, SW3.1 (A)
- net BTN_B: now reaches U3.51 (PC10)
- net BTN_B: now also R48.2, SW5.1 (A)
- net BTN_C: now reaches U3.52 (PC11)
- net BTN_C: now also R49.2, SW6.1 (A)
- net BTN_D: now reaches U3.53 (PC12)
- net BTN_D: now also R50.2, SW7.1 (A)
- new net: J10.2 (Pin_2), R44.1
- new net: R45.2, R46.2, U22.8 (Rs)
- new net CANH: J10.1 (Pin_1), J9.1 (Pin_1), U22.7 (CANH)
- new net CANL: J9.2 (Pin_2), R44.2, U22.6 (CANL)
- no-connect marks 18 -> 9
Other:
- note added: "Connectivity"
- note added: "MCU"
- note added: "Mechanical"
- note added: "Power cascade"
- note added: "Synchronous converters"
- note added: "TIM3 enc mode"
- note added: "Temperature sensors"
- note added: "User interface"
- moved on the sheet: C1, C10, C11, C12, C13, C14, C16, C17, C18, C2, C20, C21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

Commit message: Schematics seems finished, starting PCB design
Parts:
- J1: Availability Not in stock -> (none)
- J9: footprint (none) -> Connector_Phoenix_MC:PhoenixContact_MC_1,5_2-G-3.81_1x02_P3.81mm_Horizontal
Changed lines of the file:
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@@
 			)
 		)
-		(property "Footprint" ""
+		(property "Footprint" "Connector_Phoenix_MC:PhoenixContact_MC_1,5_2-G-3.81_1x02_P3.81mm_Horizontal"
 			(at 506.73 74.93 0)
 			(effects
@@
 			)
 		)
-		(property "Availability" "Not in stock"
+		(property "Availability" ""
 			(at 39.37 59.69 0)
 			(effects
