File: OchlastaPCB/_autosave-OchlastaPCB.kicad_pcb (KiCad board)
At the start: 4 copper layers, 175.1 x 89.9 mm, 139 parts, among them J1 XT60PW-M, J2 5V, J3 Conn_01x02_Socket, Q1 IRFH7440, Q2 IRFH7440, U1 AP64501SP-13, U10 INA333xxDGK, U11 INA333xxDGK, U12 INA333xxDGK, U13 UCC27282DR, U14 AP64501SP-13, U2 AP3429, U3 STM32F334R8Tx, U4 INA333xxDGK, U5 TPS7A4901DGNR, U6 INA333xxDGK, U7 INA333xxDGK, U8 INA333xxDGK, U9 INA333xxDGK, Y1 Crystal_GND24

Commit message: Schematics seems finished, starting PCB design
Parts:
- removed the C15 at (226.6, 28.4)
- removed the C15 at (221.6, 20.8)
- removed the C16 at (118.9, 108.8)
- removed the C16 at (81.8, 86.8)
- removed the L3 at (186.5, 124.0)
- removed the L3 at (112.0, 40.1)
- added C15: 100 n, Capacitor_SMD:C_0603_1608Metric, F.Cu at (395.9, 98.8)
- added C16: 10n, Capacitor_SMD:C_0603_1608Metric, F.Cu at (395.9, 101.3)
- added C45: 100 n, Capacitor_SMD:C_0603_1608Metric, F.Cu at (399.9, 113.9)
- added C46: 1 u, Capacitor_SMD:C_0603_1608Metric, F.Cu at (399.9, 116.4)
- added C47: 100 n, Capacitor_SMD:C_0603_1608Metric, F.Cu at (403.9, 81.3)
- added C48: 10 uF 50V, Capacitor_SMD:C_1206_3216Metric, F.Cu at (402.4, 165.9)
- added C49: 10 uF 50V, Capacitor_SMD:C_1206_3216Metric, F.Cu at (402.4, 169.3)
- added C50: 10 uF 50V, Capacitor_SMD:C_1206_3216Metric, F.Cu at (408.0, 155.9)
- added C51: 10 uF 50V, Capacitor_SMD:C_1206_3216Metric, F.Cu at (408.0, 159.2)
- added C52: 100 n, Capacitor_SMD:C_0603_1608Metric, F.Cu at (403.9, 83.8)
- added C53: 100 n, Capacitor_SMD:C_0603_1608Metric, F.Cu at (403.9, 86.3)
- added C54: 1 u, Capacitor_SMD:C_0603_1608Metric, F.Cu at (403.9, 88.8)
- added C55: 1 u, Capacitor_SMD:C_0603_1608Metric, F.Cu at (403.9, 91.3)
- added C56: 100 n, Capacitor_SMD:C_0603_1608Metric, F.Cu at (403.9, 93.8)
- added C57: 100 n, Capacitor_SMD:C_0603_1608Metric, F.Cu at (403.9, 96.3)
- added C58: 10 uF 50V, Capacitor_SMD:C_1206_3216Metric, F.Cu at (408.0, 162.6)
- added C59: 10 uF 50V, Capacitor_SMD:C_1206_3216Metric, F.Cu at (408.0, 165.9)
- added C60: 10 uF 50V, Capacitor_SMD:C_1206_3216Metric, F.Cu at (408.0, 169.3)
- added C61: 10 uF 50V, Capacitor_SMD:C_1206_3216Metric, F.Cu at (413.7, 155.9)
- added C62: 10 uF 50V, Capacitor_SMD:C_1206_3216Metric, F.Cu at (413.7, 159.2)
- added C63: 10 uF 50V, Capacitor_SMD:C_1206_3216Metric, F.Cu at (413.7, 162.6)
- added C64: 10 uF 50V, Capacitor_SMD:C_1206_3216Metric, F.Cu at (413.7, 165.9)
- added C65: 10 uF 50V, Capacitor_SMD:C_1206_3216Metric, F.Cu at (413.7, 169.3)
- added C66: 100 n, Capacitor_SMD:C_0603_1608Metric, F.Cu at (403.9, 98.8)
- added C67: 100 n, Capacitor_SMD:C_0603_1608Metric, F.Cu at (403.9, 101.3)
- added C68: 100 n, Capacitor_SMD:C_0603_1608Metric, F.Cu at (403.9, 103.9)
- added C69: 100 n, Capacitor_SMD:C_0603_1608Metric, F.Cu at (403.9, 106.4)
- added C70: 100 n, Capacitor_SMD:C_0603_1608Metric, F.Cu at (403.9, 108.9)
- added C71: 100 n, Capacitor_SMD:C_0603_1608Metric, F.Cu at (403.9, 111.4)
- added C72: 100 n, Capacitor_SMD:C_0603_1608Metric, F.Cu at (403.9, 113.9)
- added C73: 100 n, Capacitor_SMD:C_0603_1608Metric, F.Cu at (403.9, 116.4)
- added C74: 100 n, Capacitor_SMD:C_0603_1608Metric, F.Cu at (408.0, 81.3)
- added C75: 100 n, Capacitor_SMD:C_0603_1608Metric, F.Cu at (408.0, 83.8)
- added CP4: 100 uF, Capacitor_SMD:CP_Elec_8x10, F.Cu at (436.1, 130.8)
- added CP5: 100 uF, Capacitor_SMD:CP_Elec_8x10, F.Cu at (436.1, 140.6)
- added CP6: 100 uF, Capacitor_SMD:CP_Elec_8x10, F.Cu at (436.1, 150.5)
- added D10: SS14, Diode_SMD:D_SMA, F.Cu at (454.0, 112.2)
- added D11: SS14, Diode_SMD:D_SMA, F.Cu at (454.0, 116.8)
- added D12: SS14, Diode_SMD:D_SMA, F.Cu at (454.0, 121.3)
- added D13: SS14, Diode_SMD:D_SMA, F.Cu at (462.1, 98.6)
- added D14: SS14, Diode_SMD:D_SMA, F.Cu at (462.1, 103.1)
- added D15: SS14, Diode_SMD:D_SMA, F.Cu at (462.1, 107.7)
- added D16: SS14, Diode_SMD:D_SMA, F.Cu at (462.1, 112.2)
- added D5: SS14, Diode_SMD:D_SMA, F.Cu at (445.9, 116.8)
- added D6: SS14, Diode_SMD:D_SMA, F.Cu at (445.9, 121.3)
- added D7: SS14, Diode_SMD:D_SMA, F.Cu at (454.0, 98.6)
- added D8: SS14, Diode_SMD:D_SMA, F.Cu at (454.0, 103.1)
- added D9: SS14, Diode_SMD:D_SMA, F.Cu at (454.0, 107.7)
- added H1: MountingHole_Pad, MountingHole:MountingHole_3.2mm_M3_Pad_Via, F.Cu at (470.1, 45.6)
- added H2: MountingHole_Pad, MountingHole:MountingHole_3.2mm_M3_Pad_Via, F.Cu at (470.1, 53.6)
- added H3: MountingHole_Pad, MountingHole:MountingHole_3.2mm_M3_Pad_Via, F.Cu at (470.1, 61.5)
- added H4: MountingHole_Pad, MountingHole:MountingHole_3.2mm_M3_Pad_Via, F.Cu at (470.1, 69.5)
- added J10: CAN term jmp, Connector_PinHeader_2.54mm:PinHeader_1x02_P2.54mm_Vertical, F.Cu at (481.0, 69.8)
- added J4: Conn_01x02_Socket, TerminalBlock_WAGO:TerminalBlock_WAGO_236-402_1x02_P5.00mm_45Degree, F.Cu at (38.5, 97.1)
- added J5: Conn_01x02_Socket, TerminalBlock_WAGO:TerminalBlock_WAGO_236-402_1x02_P5.00mm_45Degree, F.Cu at (38.5, 110.9)
- added J6: Conn_01x02_Socket, TerminalBlock_WAGO:TerminalBlock_WAGO_236-402_1x02_P5.00mm_45Degree, F.Cu at (38.5, 124.6)
- added J7: Debug, Connector_IDC:IDC-Header_2x05_P2.54mm_Vertical, F.Cu at (121.9, 19.6)
- added J8: UART, Connector_PinHeader_2.54mm:PinHeader_1x03_P2.54mm_Vertical, F.Cu at (418.8, 165.4)
- added J9: CAN, Connector_Phoenix_MC:PhoenixContact_MC_1,5_2-G-3.81_1x02_P3.81mm_Horizontal, F.Cu at (97.4, 25.8)
- added L3: 22 uH, Inductor_SMD:L_APV_APH1770, F.Cu at (77.0, 89.9)
- added L5: 22 uH, Inductor_SMD:L_APV_APH1770, F.Cu at (384.0, 108.2)
- added L6: 22 uH, Inductor_SMD:L_APV_APH1770, F.Cu at (384.0, 127.0)
- added L7: 22 uH, Inductor_SMD:L_APV_APH1770, F.Cu at (384.0, 145.8)
- added Q3: IRFH7440, SnapMagic_downloads:PQFN_5x6_FET, F.Cu at (446.3, 140.2)
- added Q4: IRFH7440, SnapMagic_downloads:PQFN_5x6_FET, F.Cu at (446.3, 146.9)
- added Q5: IRFH7440, SnapMagic_downloads:PQFN_5x6_FET, F.Cu at (446.3, 153.5)
- added Q6: IRFH7440, SnapMagic_downloads:PQFN_5x6_FET, F.Cu at (454.9, 126.9)
- added Q7: IRFH7440, SnapMagic_downloads:PQFN_5x6_FET, F.Cu at (454.9, 133.6)
- added Q8: IRFH7440, SnapMagic_downloads:PQFN_5x6_FET, F.Cu at (454.9, 140.2)
- added R20: 10 R, Resistor_SMD:R_0603_1608Metric, F.Cu at (412.0, 96.3)
- added R21: 10 R, Resistor_SMD:R_0603_1608Metric, F.Cu at (412.0, 98.8)
- added R22: 10 R, Resistor_SMD:R_0603_1608Metric, F.Cu at (412.0, 101.3)
- added R23: 10 R, Resistor_SMD:R_0603_1608Metric, F.Cu at (412.0, 103.9)
- added R24: 10 R, Resistor_SMD:R_0603_1608Metric, F.Cu at (412.0, 106.4)
- added R25: 10 R, Resistor_SMD:R_0603_1608Metric, F.Cu at (412.0, 108.9)
- added R26: 10 R, Resistor_SMD:R_0603_1608Metric, F.Cu at (412.0, 111.4)
- added R27: 10 R, Resistor_SMD:R_0603_1608Metric, F.Cu at (412.0, 113.9)
- added R28: 10 R, Resistor_SMD:R_0603_1608Metric, F.Cu at (412.0, 116.4)
- added R29: 10 R, Resistor_SMD:R_0603_1608Metric, F.Cu at (416.0, 81.3)
- added R30: 10 R, Resistor_SMD:R_0603_1608Metric, F.Cu at (416.0, 83.8)
- added R31: 10 R, Resistor_SMD:R_0603_1608Metric, F.Cu at (416.0, 86.3)
- added R32: 10k, Resistor_SMD:R_0603_1608Metric, F.Cu at (416.0, 88.8)
- added R33: 10k, Resistor_SMD:R_0603_1608Metric, F.Cu at (416.0, 91.3)
- added R34: 200k 1%, Resistor_SMD:R_0603_1608Metric, F.Cu at (83.3, 134.9)
- added R35: 22.1 k 1%, Resistor_SMD:R_0603_1608Metric, F.Cu at (114.9, 121.0)
- added R36: 200k 1%, Resistor_SMD:R_0603_1608Metric, F.Cu at (416.0, 98.8)
- added R37: 22.1 k 1%, Resistor_SMD:R_0603_1608Metric, F.Cu at (416.0, 101.3)
- added R38: 200k 1%, Resistor_SMD:R_0603_1608Metric, F.Cu at (416.0, 103.9)
- added R39: 22.1 k 1%, Resistor_SMD:R_0603_1608Metric, F.Cu at (416.0, 106.4)
- added R40: 200k 1%, Resistor_SMD:R_0603_1608Metric, F.Cu at (416.0, 108.9)
- added R41: 22.1 k 1%, Resistor_SMD:R_0603_1608Metric, F.Cu at (416.0, 111.4)
- added R42: 200k 1%, Resistor_SMD:R_0603_1608Metric, F.Cu at (416.0, 113.9)
- added R43: 22.1 k 1%, Resistor_SMD:R_0603_1608Metric, F.Cu at (416.0, 116.4)
- added R44: 120 R, Resistor_SMD:R_0603_1608Metric, F.Cu at (420.0, 81.3)
- added R45: 120 R / DNP, Resistor_SMD:R_0603_1608Metric, F.Cu at (420.0, 83.8)
- added R46: DNP / 120 R, Resistor_SMD:R_0603_1608Metric, F.Cu at (420.0, 86.3)
- added R47: 10 k, Resistor_SMD:R_0603_1608Metric, F.Cu at (420.0, 88.8)
- added R48: 10 k, Resistor_SMD:R_0603_1608Metric, F.Cu at (420.0, 91.3)
- added R49: 10 k, Resistor_SMD:R_0603_1608Metric, F.Cu at (420.0, 93.8)
- added R50: 10 k, Resistor_SMD:R_0603_1608Metric, F.Cu at (420.0, 96.3)
- added R51: 10 k, Resistor_SMD:R_0603_1608Metric, F.Cu at (420.0, 98.8)
- added R52: 10 k, Resistor_SMD:R_0603_1608Metric, F.Cu at (420.0, 101.3)
- added R53: 10 k, Resistor_SMD:R_0603_1608Metric, F.Cu at (420.0, 103.9)
- added R54: 10 k, Resistor_SMD:R_0603_1608Metric, F.Cu at (420.0, 106.4)
- added R55: 10 k, Resistor_SMD:R_0603_1608Metric, F.Cu at (420.0, 108.9)
- added Rshunt1: 5 mR, Resistor_SMD:R_1206_3216Metric, F.Cu at (88.5, 144.1)
- added Rshunt2: 5 mR, Resistor_SMD:R_1206_3216Metric, F.Cu at (481.7, 166.1)
- added Rshunt3: 5 mR, Resistor_SMD:R_1206_3216Metric, F.Cu at (481.7, 169.4)
- added Rshunt4: 5 mR, Resistor_SMD:R_1206_3216Metric, F.Cu at (481.7, 172.7)
- added SW1: SW_RESET, OchlastaFootprints:SW_Push_SPST_CheapAtJLC, F.Cu at (419.8, 156.4)
- added SW2: SW_BOOT, OchlastaFootprints:SW_Push_SPST_CheapAtJLC, F.Cu at (419.8, 160.9)
- added SW3: BTN_A, Button_Switch_THT:SW_PUSH_6mm, F.Cu at (461.0, 125.6)
- added SW4: RotaryEncoder_Switch, Rotary_Encoder:RotaryEncoder_Alps_EC11E-Switch_Vertical_H20mm, F.Cu at (468.1, 101.4)
- added SW5: BTN_B, Button_Switch_THT:SW_PUSH_6mm, F.Cu at (461.0, 134.2)
- added SW6: BTN_C, Button_Switch_THT:SW_PUSH_6mm, F.Cu at (461.0, 142.7)
- added SW7: BTN_D, Button_Switch_THT:SW_PUSH_6mm, F.Cu at (461.0, 151.3)
- added SW8: BTN_L, Button_Switch_THT:SW_PUSH_6mm, F.Cu at (461.0, 159.8)
- added SW9: BTN_R, Button_Switch_THT:SW_PUSH_6mm, F.Cu at (461.0, 168.4)
- added U15: UCC27282DR, SnapMagic_downloads:SOIC127P599X175-8N, F.Cu at (478.9, 51.3)
- added U16: UCC27282DR, SnapMagic_downloads:SOIC127P599X175-8N, F.Cu at (478.9, 57.8)
- added U17: UCC27282DR, SnapMagic_downloads:SOIC127P599X175-8N, F.Cu at (478.9, 64.3)
- added U18: INA240A2D, Package_SO:SOIC-8_3.9x4.9mm_P1.27mm, F.Cu at (127.1, 155.5)
- added U19: INA240A2D, Package_SO:SOIC-8_3.9x4.9mm_P1.27mm, F.Cu at (442.5, 51.6)
- added U20: INA240A2D, Package_SO:SOIC-8_3.9x4.9mm_P1.27mm, F.Cu at (442.5, 58.2)
- added U21: INA240A2D, Package_SO:SOIC-8_3.9x4.9mm_P1.27mm, F.Cu at (442.5, 64.8)
- added U22: SN65HVD230, Package_SO:SOIC-8_3.9x4.9mm_P1.27mm, F.Cu at (442.5, 71.3)
- U5: value TPS7A4901DGNR -> TPS7A4901DGNR_Trafo_Edit
- moved C21 391.7 mm to (485.3, 58.2)
- moved C36 391.7 mm to (485.3, 61.2)
- moved C37 391.7 mm to (485.3, 64.2)
- moved L4 357.2 mm to (457.0, 72.5)
- moved U10 340.8 mm to (450.4, 67.3)
- moved U11 340.8 mm to (450.4, 71.9)
- moved U12 340.8 mm to (450.4, 76.6)
- moved U6 340.8 mm to (450.4, 48.7)
- moved U7 340.8 mm to (450.4, 53.3)
- moved U8 340.8 mm to (450.4, 58.0)
- moved U9 340.8 mm to (450.4, 62.6)
- moved U14 328.3 mm to (474.7, 171.2)
- moved U5 313.2 mm to (425.5, 165.4)
- moved Ra4 295.8 mm to (424.0, 81.3)
- moved Ra5 295.8 mm to (424.0, 83.8)
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Connections:
- C17 pad 1: Net-(C17-Pad1) -> /HSE_OUT
- C41 pad 1: Net-(J3-Pin_2) -> Net-(U18-+)
- C42 pad 1: Net-(J3-Pin_2) -> Net-(U18-+)
- C43 pad 1: Net-(J3-Pin_2) -> Net-(U18-+)
- C44 pad 1: Net-(J3-Pin_2) -> Net-(U18-+)
- CP3 pad 1: Net-(J3-Pin_2) -> Net-(U18-+)
- R8 pad 1: unconnected-(R8-Pad1) -> /HSE_IN
- TFT1 pad 3: unconnected-(TFT1-SCL-Pad3) -> /SPI_SCK
- TFT1 pad 4: unconnected-(TFT1-SDA/MOSI-Pad4) -> /SPI_MOSI
- TFT1 pad 5: unconnected-(TFT1-RST-Pad5) -> /PB10_Disp_RST
- TFT1 pad 6: unconnected-(TFT1-DC-Pad6) -> /PB11_Disp_DC
- TFT1 pad 7: unconnected-(TFT1-CS-Pad7) -> /PB9_Disp_CS
- U3 pad 1: unconnected-(U3-VBAT-Pad1) -> +3V3
- U3 pad 10: unconnected-(U3-PC2-Pad10) -> /U_out_3
- U3 pad 11: unconnected-(U3-PC3-Pad11) -> /temp_U_out_1
- U3 pad 12: unconnected-(U3-VSSA-Pad12) -> GND
- U3 pad 13: unconnected-(U3-VDDA-Pad13) -> +3.3VA
- U3 pad 14: unconnected-(U3-PA0-Pad14) -> /I_out_1
- U3 pad 15: unconnected-(U3-PA1-Pad15) -> /I_out_2
- U3 pad 16: unconnected-(U3-PA2-Pad16) -> /I_out_3
- U3 pad 17: unconnected-(U3-PA3-Pad17) -> /I_out_4
- U3 pad 18: Net-(U3-VSS-Pad18) -> GND
- U3 pad 19: unconnected-(U3-VDD-Pad19) -> +3V3
- U3 pad 2: unconnected-(U3-PC13-Pad2) -> /BTN_L
- U3 pad 20: unconnected-(U3-PA4-Pad20) -> /temp_U_out_2
- U3 pad 21: unconnected-(U3-PA5-Pad21) -> /temp_U_out_3
- U3 pad 22: unconnected-(U3-PA6-Pad22) -> /temp_U_out_4
- U3 pad 23: unconnected-(U3-PA7-Pad23) -> /temp_U_out_5
- U3 pad 24: unconnected-(U3-PC4-Pad24) -> /temp_U_out_6
- U3 pad 25: unconnected-(U3-PC5-Pad25) -> /temp_U_out_7
- U3 pad 26: unconnected-(U3-PB0-Pad26) -> /U_out_4
- U3 pad 27: unconnected-(U3-PB1-Pad27) -> /U_input_div
- U3 pad 28: unconnected-(U3-PB2-Pad28) -> /temp_U_out_8
- U3 pad 29: unconnected-(U3-PB10-Pad29) -> /PB10_Disp_RST
- U3 pad 3: unconnected-(U3-PC14-Pad3) -> /BTN_R
- U3 pad 30: unconnected-(U3-PB11-Pad30) -> /PB11_Disp_DC
- U3 pad 31: Net-(U3-VSS-Pad18) -> GND
- U3 pad 32: unconnected-(U3-VDD-Pad32) -> +3V3
- U3 pad 33: unconnected-(U3-PB12-Pad33) -> /HRTIM_C_Hi
- U3 pad 34: unconnected-(U3-PB13-Pad34) -> /HRTIM_C_Lo
- U3 pad 35: unconnected-(U3-PB14-Pad35) -> /HRTIM_D_Hi
- U3 pad 36: unconnected-(U3-PB15-Pad36) -> /HRTIM_D_Lo
- U3 pad 37: unconnected-(U3-PC6-Pad37) -> /ENC_A
- U3 pad 38: unconnected-(U3-PC7-Pad38) -> /ENC_B
- U3 pad 39: unconnected-(U3-PC8-Pad39) -> /BTN_ENC
- U3 pad 40: unconnected-(U3-PC9-Pad40) -> /BTN_A
- U3 pad 41: unconnected-(U3-PA8-Pad41) -> /HRTIM_A_Hi
- U3 pad 42: unconnected-(U3-PA9-Pad42) -> /HRTIM_A_Lo
- U3 pad 43: unconnected-(U3-PA10-Pad43) -> /HRTIM_B_Hi
- U3 pad 44: unconnected-(U3-PA11-Pad44) -> /HRTIM_B_Lo
- U3 pad 45: unconnected-(U3-PA12-Pad45) -> /CAN_TX
- U3 pad 46: unconnected-(U3-PA13-Pad46) -> /SWDIO
- U3 pad 47: Net-(U3-VSS-Pad18) -> GND
- U3 pad 48: unconnected-(U3-VDD-Pad48) -> +3V3
- U3 pad 49: unconnected-(U3-PA14-Pad49) -> /SWCLK
- U3 pad 5: unconnected-(U3-PF0-Pad5) -> /HSE_IN
- U3 pad 51: unconnected-(U3-PC10-Pad51) -> /BTN_B
- U3 pad 52: unconnected-(U3-PC11-Pad52) -> /BTN_C
- U3 pad 53: unconnected-(U3-PC12-Pad53) -> /BTN_D
- U3 pad 55: unconnected-(U3-PB3-Pad55) -> /SPI_SCK
- U3 pad 56: unconnected-(U3-PB4-Pad56) -> /SPI_MISO
- U3 pad 57: unconnected-(U3-PB5-Pad57) -> /SPI_MOSI
- U3 pad 58: unconnected-(U3-PB6-Pad58) -> /UART_TX
- U3 pad 59: unconnected-(U3-PB7-Pad59) -> /UART_RX
- U3 pad 6: unconnected-(U3-PF1-Pad6) -> /HSE_OUT
- U3 pad 60: unconnected-(U3-BOOT0-Pad60) -> /BOOT0
- U3 pad 61: unconnected-(U3-PB8-Pad61) -> /CAN_RX
- U3 pad 62: unconnected-(U3-PB9-Pad62) -> /PB9_Disp_CS
- U3 pad 63: Net-(U3-VSS-Pad18) -> GND
- U3 pad 64: unconnected-(U3-VDD-Pad64) -> +3V3
- U3 pad 7: unconnected-(U3-NRST-Pad7) -> /NRST
- U3 pad 8: unconnected-(U3-PC0-Pad8) -> /U_out_1
- U3 pad 9: unconnected-(U3-PC1-Pad9) -> /U_out_2
- Y1 pad 1: Net-(C17-Pad1) -> /HSE_OUT
Routing:
- net Net-(U4-+): track 14.4 -> 0.00 mm
- net GND: track 11.3 -> 0.00 mm
- net +3V3: track 10.7 -> 0.00 mm, vias 1 -> 0
- net Net-(U4--): track 8.31 -> 0.00 mm
- net +5V: track 5.94 -> 0.00 mm
- net Net-(U1-COMP): track 2.40 -> 0.00 mm
- net Net-(U1-SW): track 0.00 -> 2.38 mm
- net Net-(U1-BST): track 0.00 -> 2.38 mm
- net Net-(C5-Pad1): track 1.32 -> 0.00 mm
Other:
- board size 175.1 x 89.9 mm -> 60.5 x 30.5 mm
